Commit message: fixed lidar bugs and created new world

File: sanad_ws/src/sanad_description/urdf/lidar.xacro (robot description, xacro)
@@ -4,8 +4,15 @@
   <xacro:property name="lidar_radius" value="0.1" />
   <xacro:property name="lidar_height" value="0.05" />
-    <!-- System plugin for all sensors -->
+    <!-- System plugin for all sensors
     <plugin filename="libignition-gazebo-sensors-system.so" name="ignition::gazebo::systems::Sensors">
       <render_engine>ogre</render_engine>
-    </plugin>
+    </plugin> -->
+  <!-- Lidar joint -->
+  <joint name="base_lidar_joint" type="fixed">
+    <!-- Position = front of base, at same height as camera or lower -->
+    <origin xyz="0.0 0.0 0.25" rpy="0.0 0.0 0.0"/>
+    <parent link="base_link"/>
+    <child link="lidar_link"/>
+  </joint>
   <!-- Lidar link -->
   <link name="lidar_link">
@@ -22,22 +29,16 @@
     </collision>
   </link>
-  <!-- Lidar joint -->
-  <joint name="base_lidar_joint" type="fixed">
-    <!-- Position = front of base, at same height as camera or lower -->
-    <origin xyz="0.0 0.0 0.25" rpy="0.0 0.0 0.0"/>
-    <parent link="base_link"/>
-    <child link="lidar_link"/>
-  </joint>
   <!-- Gazebo Lidar Plugin -->
   <gazebo reference="lidar_link">
-    <sensor name="lidar" type="gpu_ray">
+    <material>Gazebo/Black</material>
+    <sensor name="lidar" type="gpu_lidar">
       <pose>0 0 0 0 0 0</pose>
       <visualize>true</visualize>
       <update_rate>10</update_rate>
-      <ray>
+      <lidar>
         <scan>
           <horizontal>
             <samples>360</samples>
-            <resolution>1</resolution>
+            <!-- <resolution>1</resolution> -->
             <min_angle>-3.14</min_angle>
             <max_angle>3.14</max_angle>
@@ -48,7 +49,8 @@
           <max>12</max>
         </range>
-      </ray>
+      </lidar>
       <topic>lidar/scan</topic>
-      <always_on>1</always_on>
+      <!-- <always_on>1</always_on> -->
+      <gz_frame_id>lidar_link</gz_frame_id>
     </sensor>
   </gazebo>
