Commit message: added ros2_control intial files

File: sanad_ws/src/sanad_description/urdf/mobile_base.xacro (robot description, xacro)
@@ -86,5 +86,5 @@
     <axis xyz="0 0 1" />
   </joint>
-  <joint name="base_caster_wheel_joint" type="continuous">
+  <joint name="base_caster_wheel_joint" type="fixed">
     <parent link="base_link" />
     <child link="caster_wheel_link" />

File: sanad_ws/src/sanad_description/urdf/sanad.urdf.xacro (robot description, xacro)
@@ -2,4 +2,5 @@
 <robot name="sanad" xmlns:xacro="http://www.ros.org/wiki/xacro">
   <xacro:include filename="common_properties.xacro"/>
+  <xacro:include filename="mobile_base.ros2_control.xacro"/>
   <xacro:include filename="mobile_base.xacro"/>
   <xacro:include filename="mobile_base_gazebo.xacro"/>
