Commit message: added gazebo to ros2 bridge

File: sanad_ws/src/sanad_description/urdf/mobile_base.ros2_control.xacro (robot description, xacro)
@@ -3,6 +3,7 @@
   <ros2_control name="MobileBaseHardwareInterface" type="system">
     <hardware>
-      <plugin>mock_components/GenericSystem</plugin>
-      <param name="calculate_dynamics">true</param>
+      <!-- <plugin>mock_components/GenericSystem</plugin>
+      <param name="calculate_dynamics">true</param> -->
+      <plugin>gz_ros2_control/GazeboSimSystem</plugin>
     </hardware>
     <joint name="base_left_wheel_joint">
@@ -10,10 +11,10 @@
         <state_interface name="position"/>
         <state_interface name="velocity"/>
-      </joint>
-      <joint name="base_right_wheel_joint">
-        <command_interface name="velocity"/>
-        <state_interface name="position"/>
-        <state_interface name="velocity"/>
-      </joint>
+    </joint>
+    <joint name="base_right_wheel_joint">
+      <command_interface name="velocity"/>
+      <state_interface name="position"/>
+      <state_interface name="velocity"/>
+    </joint>
   </ros2_control>
 </robot>

File: sanad_ws/src/sanad_description/urdf/mobile_base_gazebo.xacro (robot description, xacro)
@@ -6,5 +6,5 @@
   </gazebo>
 <gazebo>
-<plugin filename="gz-sim-diff-drive-system"
+  <plugin filename="gz-sim-diff-drive-system"
       name="gz::sim::systems::DiffDrive">
       <left_joint>base_left_wheel_joint</left_joint>
@@ -25,3 +25,8 @@
     </plugin>
   </gazebo>
+  <gazebo>
+    <plugin filename="gz_ros2_control-system" name="gz_ros2_control::GazeboSimROS2ControlPlugin">
+      <parameters>$(find sanad_bringup)/config/sanad_controllers.yaml</parameters>
+    </plugin>
+  </gazebo>
 </robot>

Commit message: Enhance hardware interface support by adding ros2_control_hardware parameter for Gazebo, real, and mock hardware configurations

File: sanad_ws/src/sanad_description/urdf/mobile_base.ros2_control.xacro (robot description, xacro)
@@ -3,11 +3,13 @@
   <ros2_control name="diffbot_ros2_control" type="system">
     <hardware>
-      <!-- ^mock components for testing purposes -->
-      <!-- <plugin>mock_components/GenericSystem</plugin>
-      <param name="calculate_dynamics">true</param> -->
-      <!-- ^gz-sim integration -->
-      <!-- <plugin>gz_ros2_control/GazeboSimSystem</plugin> -->
-      <!-- ^diffdrive arduino hardware interface -->
-      <plugin>diffdrive_arduino/DiffDriveArduinoHardware</plugin>
+      <xacro:if value="${ros2_control_hardware == 'mock'}">
+        <plugin>mock_components/GenericSystem</plugin>
+        <param name="calculate_dynamics">true</param>
+      </xacro:if>
+      <xacro:if value="${ros2_control_hardware == 'gazebo'}">
+        <plugin>gz_ros2_control/GazeboSimSystem</plugin>
+      </xacro:if>
+      <xacro:unless value="${ros2_control_hardware == 'mock' or ros2_control_hardware == 'gazebo'}">
+        <plugin>diffdrive_arduino/DiffDriveArduinoHardware</plugin>
       <param name="left_wheel_name">base_left_wheel_joint</param>
       <param name="right_wheel_name">base_right_wheel_joint</param>
@@ -21,4 +23,5 @@
       <param name="pid_i">0</param>
       <param name="pid_o">50</param>
+      </xacro:unless>
     </hardware>
     <joint name="base_left_wheel_joint">

File: sanad_ws/src/sanad_description/urdf/sanad.urdf.xacro (robot description, xacro)
@@ -1,4 +1,5 @@
 <?xml version="1.0"?>
 <robot name="sanad" xmlns:xacro="http://www.ros.org/wiki/xacro">
+  <xacro:property name="ros2_control_hardware" value="$(arg ros2_control_hardware)" />
   <xacro:include filename="common_properties.xacro"/>
   <xacro:include filename="mobile_base.xacro"/>
