Commit message: return to old code

File: src/sanad_description/urdf/sanad_ros2_control.xacro (robot description, xacro)
@@ -1,32 +1,29 @@
 <?xml version="1.0"?>
-<robot xmlns:xacro="http://www.ros.org/wiki/xacro">
-    <ros2_control name="sanad_ros2_control" type="system">
-        <hardware>
-            <xacro:if value="$(arg is_sim)">
-                <!-- ROS 2 Humble -->
-                <xacro:if value="$(arg is_ignition)">
-                        <plugin>ign_ros2_control/IgnitionSystem</plugin>
-                </xacro:if>
-                <!-- ROS 2 Iron or above -->
-                <xacro:unless value="$(arg is_ignition)">
-                        <plugin>gz_ros2_control/GazeboSimSystem</plugin>
-                </xacro:unless>
+<robot xmlns:xacro="http://www.ros.org/wiki/xacro" name="sanad">
+    <ros2_control name="RobotSystem" type="system">
+        <!-- ros2_control Gazebo -->
+        <xacro:if value="$(arg is_sim)">
+            <!-- ROS 2 Humble -->
+            <xacro:if value="$(arg is_ignition)">
+                <hardware>
+                    <plugin>ign_ros2_control/IgnitionSystem</plugin>
+                </hardware>
             </xacro:if>
-            <xacro:unless value="$(arg is_sim)">
-                <plugin>diffdrive_arduino/DiffDriveArduinoHardware</plugin>
-                <param name="left_wheel_name">wheel_left_joint</param>
-                <param name="right_wheel_name">wheel_right_joint</param>
-                <param name="loop_rate">30</param>
-                <param name="device">/dev/serial/by-path/platform-fd500000.pcie-pci-0000:01:00.0-usb-0:1.3:1.0-port0</param>
-                <param name="baud_rate">57600</param>
-                <param name="timeout_ms">1000</param>
-                <param name="enc_counts_per_rev">3436</param>
-                <param name="pid_p">20</param>
-                <param name="pid_d">12</param>
-                <param name="pid_i">0</param>
-                <param name="pid_o">50</param>
+            <!-- ROS 2 Iron or above -->
+            <xacro:unless value="$(arg is_ignition)">
+                <hardware>
+                    <plugin>gz_ros2_control/GazeboSimSystem</plugin>
+                </hardware>
             </xacro:unless>
-        </hardware>
-                <joint name="wheel_left_joint">
+        </xacro:if>
+        <!-- ros2_control Real Robot -->
+        <xacro:unless value="$(arg is_sim)">
+            <hardware>
+                <plugin>sanad_firmware/SanadInterface</plugin>
+                <param name="port">/dev/ttyUSB0</param>
+            </hardware>
+        </xacro:unless>
+        <!-- ros2_control Common Interfaces -->
+        <joint name="wheel_left_joint">
             <command_interface name="velocity">
               <param name="min">-1</param>
