Commit message: restructure code

File: src/sanad_description/urdf/sanad.urdf.xacro (robot description, xacro)
@@ -1,10 +1,218 @@
 <?xml version="1.0"?>
-<robot name="sanad" xmlns:xacro="http://www.ros.org/wiki/xacro">
-  <xacro:property name="ros2_control_hardware" value="$(arg ros2_control_hardware)" />
-  <xacro:include filename="common_properties.xacro"/>
-  <xacro:include filename="mobile_base.xacro"/>
-  <xacro:include filename="mobile_base_gazebo.xacro"/>
-  <xacro:include filename="camera.xacro"/>
-  <xacro:include filename="lidar.xacro"/>=
-  <xacro:include filename="mobile_base.ros2_control.xacro"/>
+<robot name="sanad" xmlns:xacro="http://ros.org/wiki/xacro">
+  <!-- Load Simulated or Real Hardware Interfaces -->
+  <xacro:arg name="is_sim" default="true"/>
+  <!-- Include Gazebo Parameters -->
+  <xacro:include filename="$(find sanad_description)/urdf/sanad_gazebo.xacro" />
+  <!-- Include ros2_control Plugins -->
+  <xacro:include filename="$(find sanad_description)/urdf/sanad_ros2_control.xacro" />
+  <link name="base_footprint"/>
+  <link name="base_link">
+    <inertial>
+      <origin xyz="0 0 0.04" rpy="0.0 0.25 0.3" />
+      <mass value="8.2573504e-01"/>
+      <inertia ixx="2.2124416e-02" ixy="-1.2294101e-04" ixz="3.4938785e-04"
+               iyy="2.1193702e-02" iyz="-5.0120904e-05"
+               izz="2.0064271e-02" />
+    </inertial>
+    <visual>
+      <origin xyz="0 0 0" rpy="0 0 0" />
+      <geometry>
+        <mesh filename="package://sanad_description/meshes/base_link.STL" />
+      </geometry>
+      <material name="black"/>
+    </visual>
+    <collision>
+      <origin xyz="0 0 0" rpy="0 0 0" />
+      <geometry>
+        <mesh filename="package://sanad_description/meshes/base_link.STL" />
+      </geometry>
+    </collision>
+  </link>
+  <joint name="base_joint" type="fixed">
+    <parent link="base_footprint"/>
+    <child link="base_link" />
+    <origin xyz="0 0 0.033" rpy="0 0 0"/>
+  </joint>
+  <link name="wheel_right_link">
+    <inertial>
+      <origin xyz="0 -0.014 0" rpy="0 0 0" />
+      <mass value="0.0530086090966721" />
+      <inertia ixx="1.88176298336665E-05" ixy="-4.8444933029987E-10" ixz="1.88163708851143E-08"
+               iyy="3.11510738647764E-05" iyz="-6.93560663069607E-11"
+               izz="1.8801969558182E-05" />
+    </inertial>
+    <visual>
+      <origin xyz="0 0 0" rpy="1.57 0 0" />
+      <geometry>
+        <mesh filename="package://sanad_description/meshes/wheel_right_link.STL" />
+      </geometry>
+      <material name="blue"/>
+    </visual>
+    <collision>
+      <origin xyz="0 -0.015 0" rpy="1.57 0 0" />
+      <geometry>
+        <sphere radius="0.033"/>
+      </geometry>
+    </collision>
+  </link>
+  <joint name="wheel_right_joint" type="continuous">
+    <origin xyz="0 -0.0701101849418637 0" rpy="0 0 0" />
+    <parent link="base_link" />
+    <child link="wheel_right_link" />
+    <axis xyz="0 1 0" />
+  </joint>
+  <link
+    name="wheel_left_link">
+    <inertial>
+      <origin xyz="0 0.014 0" rpy="0 0 0" />
+      <mass value="0.0530086043217644" />
+      <inertia ixx="1.8792911368909E-05"  ixy="3.31256392204584E-10" ixz="-1.14082001662767E-08"
+               iyy="3.11510738759073E-05" iyz="-3.60499245082192E-10"
+               izz="1.88266886146847E-05" />
+    </inertial>
+    <visual>
+      <origin xyz="0 0 0" rpy="-1.57 0 0" />
+      <geometry>
+        <mesh filename="package://sanad_description/meshes/wheel_left_link.STL" />
+      </geometry>
+      <material name="blue"/>
+    </visual>
+    <collision>
+      <origin xyz="0 0.015 0" rpy="-1.57 0 0" />
+      <geometry>
+        <sphere radius="0.033"/>
+      </geometry>
+    </collision>
+  </link>
+  <joint name="wheel_left_joint" type="continuous">
+    <origin xyz="0 0.0701101849418642 0" rpy="0 0 0" />
+    <parent link="base_link" />
+    <child link="wheel_left_link" />
+    <axis xyz="0 1 0" />
+  </joint>
+  <link name="caster_front_link">
+    <inertial>
+      <origin xyz="3.89968128948481E-07 2.40073004698083E-07 0.00219173397061506" rpy="0 0 0" />
+      <mass value="1.44379265037903E-06" />
+      <inertia ixx="7.23075276010246E-11" ixy="-6.10956883467859E-16" ixz="2.22849693525031E-15"
+               iyy="3.8713793085917E-11"  iyz="2.93909858781952E-15"
+               izz="1.00967486676306E-10" />
+    </inertial>
+    <visual>
+      <origin xyz="0 0 0" rpy="0 0 0" />
+      <geometry>
+        <mesh filename="package://sanad_description/meshes/caster_front_link.STL" />
+      </geometry>
+      <material name="silver"/>
+    </visual>
+    <collision>
+      <origin xyz="0 0 0" rpy="0 0 0" />
+      <geometry>
+        <sphere radius="0.005"/>
+      </geometry>
+    </collision>
+  </link>
+  <joint name="caster_front_joint" type="fixed">
+    <origin xyz="0.04755 0 -0.0275" rpy="0 0 0" />
+    <parent link="base_link" />
+    <child link="caster_front_link" />
+    <axis xyz="0 0 0" />
+  </joint>
+  <link name="caster_rear_link">
+    <inertial>
+      <origin xyz="3.8996812895542E-07 2.40073004698083E-07 0.00219173397061509" rpy="0 0 0" />
+      <mass value="1.44379265037902E-06" />
+      <inertia ixx="7.23075276010246E-11" ixy="-6.10956872363424E-16" ixz="2.22849693527207E-15"
+               iyy="3.87137930859167E-11" iyz="2.939098587861E-15"
+               izz="1.00967486676306E-10" />
+    </inertial>
+    <visual>
+      <origin xyz="0 0 0" rpy="0 0 0" />
+      <geometry>
+        <mesh filename="package://sanad_description/meshes/caster_rear_link.STL" />
+      </geometry>
+      <material name="silver"/>
+    </visual>
+    <collision>
+      <origin xyz="0 0 0" rpy="0 0 0" />
+      <geometry>
+        <sphere radius="0.005"/>
+      </geometry>
+    </collision>
+  </link>
+  <joint name="caster_rear_joint" type="fixed">
+    <origin xyz="-0.04755 0 -0.0275" rpy="0 0 0" />
+    <parent link="base_link" />
+    <child link="caster_rear_link" />
+    <axis xyz="0 0 0" />
+  </joint>
+  <link name="imu_link">
+    <inertial>
+      <origin xyz="-0.00552433659106688 0.000168210391520346 0.000514000497342681" rpy="0 0 0" />
+      <mass value="0.000528415362211671" />
+      <inertia ixx="1.46176048428261E-08" ixy="1.40015117949421E-10" ixz="-1.99633872937403E-12"
+               iyy="8.59662482954888E-09" iyz="7.52375112767959E-12"
+               izz="2.30279421279312E-08" />
+    </inertial>
+    <visual>
+      <origin xyz="0 0 0" rpy="0 0 0" />
+      <geometry>
+        <mesh filename="package://sanad_description/meshes/imu_link.STL" />
+      </geometry>
+      <material name="blue"/>
+    </visual>
+    <collision>
+      <origin xyz="0 0 0" rpy="0 0 0" />
+      <geometry>
+        <mesh filename="package://sanad_description/meshes/imu_link.STL" />
+      </geometry>
+    </collision>
+  </link>
+  <joint name="imu_joint" type="fixed">
+    <origin xyz="0 0 0.0698986241758014" rpy="0 0 0" />
+    <parent link="base_link" />
+    <child link="imu_link" />
+    <axis xyz="0 0 0" />
+  </joint>
+  <link name="laser_link">
+    <inertial>
+      <origin xyz="-0.011945780406062 -0.000381929217680526 -0.0170649378129477" rpy="0 0 0" />
+      <mass value="0.073084435549317" />
+      <inertia ixx="1.96074931730795E-05" ixy="-3.62091076640009E-07" ixz="4.28230084046735E-07"
+               iyy="2.40983835136327E-05" iyz="1.50180909250652E-08"
+               izz="4.14184164228595E-05" />
+    </inertial>
+    <visual>
+      <origin xyz="0 0 0" rpy="0 0 0" />
+      <geometry>
+        <mesh filename="package://sanad_description/meshes/laser_link.STL" />
+      </geometry>
+      <material name="dark_grey"/>
+    </visual>
+    <collision>
+      <origin xyz="0 0 0" rpy="0 0 0" />
+      <geometry>
+        <mesh filename="package://sanad_description/meshes/laser_link.STL" />
+      </geometry>
+    </collision>
+  </link>
+  <joint name="laser_joint" type="fixed">
+    <origin xyz="-0.0050526 -0.0023221 0.1208" rpy="0 0 3.14" />
+    <parent link="base_link" />
+    <child link="laser_link" />
+    <axis xyz="0 0 0" />
+  </joint>
+  <material name="blue">
+    <color rgba="0 0 1 1"/>
+  </material>
+  <material name="black">
+    <color rgba="0 0 0 1"/>
+  </material>
+  <material name="silver">
+    <color rgba="0.79 0.82 0.93 1"/>
+  </material>
+  <material name="dark_grey">
+    <color rgba="0.3 0.3 0.3 1"/>
+  </material>
 </robot>

Commit message: adding wheelchair intial urdf

File: src/sanad_description/urdf/sanad.urdf.xacro (robot description, xacro)
@@ -1,3 +1,4 @@
 <?xml version="1.0"?>
+<!-- ^fix the center of base_link -->
 <robot name="sanad" xmlns:xacro="http://ros.org/wiki/xacro">
   <!-- Load Simulated or Real Hardware Interfaces -->
@@ -19,14 +20,14 @@
     </inertial>
     <visual>
-      <origin xyz="0 0 0" rpy="0 0 0" />
-      <geometry>
-        <mesh filename="package://sanad_description/meshes/base_link.STL" />
-      </geometry>
-      <material name="black"/>
-    </visual>
-    <collision>
-      <origin xyz="0 0 0" rpy="0 0 0" />
-      <geometry>
-        <mesh filename="package://sanad_description/meshes/base_link.STL" />
+      <origin xyz="0 ${0.416/2} 0" rpy="0 0 0" />
+      <geometry>
+        <mesh filename="package://sanad_description/meshes/chase.stl" scale="0.001 0.001 0.001" />
+      </geometry>
+      <material name="silver"/>
+    </visual>
+    <collision>
+      <origin xyz="0 ${0.416/2} 0" rpy="0 0 0" />
+      <geometry>
+        <mesh filename="package://sanad_description/meshes/chase.stl" scale="0.001 0.001 0.001" />
       </geometry>
     </collision>
@@ -35,38 +36,9 @@
     <parent link="base_footprint"/>
     <child link="base_link" />
-    <origin xyz="0 0 0.033" rpy="0 0 0"/>
+    <origin xyz="0 0 0.533" rpy="0 0 0"/>
   </joint>
   <link name="wheel_right_link">
     <inertial>
-      <origin xyz="0 -0.014 0" rpy="0 0 0" />
-      <mass value="0.0530086090966721" />
-      <inertia ixx="1.88176298336665E-05" ixy="-4.8444933029987E-10" ixz="1.88163708851143E-08"
-               iyy="3.11510738647764E-05" iyz="-6.93560663069607E-11"
-               izz="1.8801969558182E-05" />
-    </inertial>
-    <visual>
-      <origin xyz="0 0 0" rpy="1.57 0 0" />
-      <geometry>
-        <mesh filename="package://sanad_description/meshes/wheel_right_link.STL" />
-      </geometry>
-      <material name="blue"/>
-    </visual>
-    <collision>
-      <origin xyz="0 -0.015 0" rpy="1.57 0 0" />
-      <geometry>
-        <sphere radius="0.033"/>
-      </geometry>
-    </collision>
-  </link>
-  <joint name="wheel_right_joint" type="continuous">
-    <origin xyz="0 -0.0701101849418637 0" rpy="0 0 0" />
-    <parent link="base_link" />
-    <child link="wheel_right_link" />
-    <axis xyz="0 1 0" />
-  </joint>
-  <link
-    name="wheel_left_link">
-    <inertial>
-      <origin xyz="0 0.014 0" rpy="0 0 0" />
+      <origin xyz="0 0 0" rpy="0 0 0" />
       <mass value="0.0530086043217644" />
       <inertia ixx="1.8792911368909E-05"  ixy="3.31256392204584E-10" ixz="-1.14082001662767E-08"
@@ -75,19 +47,48 @@
     </inertial>
     <visual>
-      <origin xyz="0 0 0" rpy="-1.57 0 0" />
-      <geometry>
-        <mesh filename="package://sanad_description/meshes/wheel_left_link.STL" />
+      <origin xyz="0 0 0" rpy="0 0 1.57" />
+      <geometry>
+        <mesh filename="package://sanad_description/meshes/Back_wheel.stl" scale="0.001 0.001 0.001" />
       </geometry>
       <material name="blue"/>
     </visual>
     <collision>
-      <origin xyz="0 0.015 0" rpy="-1.57 0 0" />
-      <geometry>
-        <sphere radius="0.033"/>
+      <origin xyz="0 0 0" rpy="0 0 0" />
+      <geometry>
+        <sphere radius="0.15875"/>
+      </geometry>
+    </collision>
+  </link>
+  <joint name="wheel_right_joint" type="continuous">
+    <origin xyz="0.22 -${0.580/2} -0.37" rpy="0 0 0" />
+    <parent link="base_link" />
+    <child link="wheel_right_link" />
+    <axis xyz="0 1 0" />
+  </joint>
+  <link
+    name="wheel_left_link">
+    <inertial>
+      <origin xyz="0 0 0" rpy="0 0 0" />
+      <mass value="0.0530086043217644" />
+      <inertia ixx="1.8792911368909E-05"  ixy="3.31256392204584E-10" ixz="-1.14082001662767E-08"
+               iyy="3.11510738759073E-05" iyz="-3.60499245082192E-10"
+               izz="1.88266886146847E-05" />
+    </inertial>
+    <visual>
+      <origin xyz="0 0 0" rpy="0 0 1.57" />
+      <geometry>
+        <mesh filename="package://sanad_description/meshes/Back_wheel.stl" scale="0.001 0.001 0.001" />
+      </geometry>
+      <material name="blue"/>
+    </visual>
+    <collision>
+      <origin xyz="0 0 0" rpy="0 0 0" />
+      <geometry>
+        <sphere radius="0.15875"/>
       </geometry>
     </collision>
   </link>
   <joint name="wheel_left_joint" type="continuous">
-    <origin xyz="0 0.0701101849418642 0" rpy="0 0 0" />
+    <origin xyz="0.22 ${0.580/2} -0.37" rpy="0 0 0" />
     <parent link="base_link" />
     <child link="wheel_left_link" />
@@ -105,5 +106,5 @@
       <origin xyz="0 0 0" rpy="0 0 0" />
       <geometry>
-        <mesh filename="package://sanad_description/meshes/caster_front_link.STL" />
+        <mesh filename="package://sanad_description/meshes/caster_wheel.stl" scale="0.001 0.001 0.001" />
       </geometry>
       <material name="silver"/>
@@ -112,10 +113,10 @@
       <origin xyz="0 0 0" rpy="0 0 0" />
       <geometry>
-        <sphere radius="0.005"/>
+        <sphere radius="0.08888"/>
       </geometry>
     </collision>
   </link>
   <joint name="caster_front_joint" type="fixed">
-    <origin xyz="0.04755 0 -0.0275" rpy="0 0 0" />
+    <origin xyz="-0.32 0.251 -0.44" rpy="1.57 1.57 0" />
     <parent link="base_link" />
     <child link="caster_front_link" />
@@ -133,5 +134,5 @@
       <origin xyz="0 0 0" rpy="0 0 0" />
       <geometry>
-        <mesh filename="package://sanad_description/meshes/caster_rear_link.STL" />
+        <mesh filename="package://sanad_description/meshes/caster_wheel.stl" scale="0.001 0.001 0.001" />
       </geometry>
       <material name="silver"/>
@@ -140,10 +141,10 @@
       <origin xyz="0 0 0" rpy="0 0 0" />
       <geometry>
-        <sphere radius="0.005"/>
+        <sphere radius="0.08888"/>
       </geometry>
     </collision>
   </link>
   <joint name="caster_rear_joint" type="fixed">
-    <origin xyz="-0.04755 0 -0.0275" rpy="0 0 0" />
+    <origin xyz="-0.32 -0.251 -0.44" rpy="1.57 1.57 0" />
     <parent link="base_link" />
     <child link="caster_rear_link" />
@@ -178,5 +179,5 @@
     <axis xyz="0 0 0" />
   </joint>
-  <link name="laser_link">
+  <link name="laser_right_link">
     <inertial>
       <origin xyz="-0.011945780406062 -0.000381929217680526 -0.0170649378129477" rpy="0 0 0" />
@@ -200,8 +201,36 @@
     </collision>
   </link>
-  <joint name="laser_joint" type="fixed">
-    <origin xyz="-0.0050526 -0.0023221 0.1208" rpy="0 0 3.14" />
-    <parent link="base_link" />
-    <child link="laser_link" />
+  <link name="laser_left_link">
+    <inertial>
+      <origin xyz="-0.011945780406062 -0.000381929217680526 -0.0170649378129477" rpy="0 0 0" />
+      <mass value="0.073084435549317" />
+      <inertia ixx="1.96074931730795E-05" ixy="-3.62091076640009E-07" ixz="4.28230084046735E-07"
+               iyy="2.40983835136327E-05" iyz="1.50180909250652E-08"
+               izz="4.14184164228595E-05" />
+    </inertial>
+    <visual>
+      <origin xyz="0 0 0" rpy="0 0 0" />
+      <geometry>
+        <mesh filename="package://sanad_description/meshes/laser_link.STL" />
+      </geometry>
+      <material name="dark_grey"/>
+    </visual>
+    <collision>
+      <origin xyz="0 0 0" rpy="0 0 0" />
+      <geometry>
+        <mesh filename="package://sanad_description/meshes/laser_link.STL" />
+      </geometry>
+    </collision>
+  </link>
+  <joint name="laser_right_joint" type="fixed">
+    <origin xyz="-0.265 ${-(0.245 +0.1)} 0.06" rpy="0 0 3.14" />
+    <parent link="base_link" />
+    <child link="laser_right_link" />
+    <axis xyz="0 0 0" />
+  </joint>
+    <joint name="laser_left_joint" type="fixed">
+    <origin xyz="-0.265 ${(0.245 +0.1)} 0.06" rpy="0 0 3.14" />
+    <parent link="base_link" />
+    <child link="laser_left_link" />
     <axis xyz="0 0 0" />
   </joint>

File: src/sanad_description/urdf/sanad_gazebo.xacro (robot description, xacro)
@@ -113,12 +113,42 @@
     </sensor>
   </gazebo>
-  <!-- 2D Laser Sensor -->
-  <gazebo reference="laser_link">
-    <sensor name="lidar" type="gpu_lidar">
+  <!-- 2D Laser Sensor - Right -->
+  <gazebo reference="laser_right_link">
+    <sensor name="lidar_right" type="gpu_lidar">
+      <always_on>true</always_on>
+      <visualize>true</visualize>
+      <topic>scan_rear</topic>
+      <update_rate>5</update_rate>
+      <gz_frame_id>laser_right_link</gz_frame_id>
+      <lidar>
+        <scan>
+          <horizontal>
+            <samples>360</samples>
+            <resolution>1.00000</resolution>
+            <min_angle>0.000000</min_angle>
+            <max_angle>6.280000</max_angle>
+          </horizontal>
+        </scan>
+        <range>
+          <min>0.120000</min>
+          <max>12.0</max>
+          <resolution>0.02</resolution>
+        </range>
+        <noise>
+          <type>gaussian</type>
+          <mean>0.0</mean>
+          <stddev>0.01</stddev>
+        </noise>
+      </lidar>
+    </sensor>
+  </gazebo>
+  <!-- 2D Laser Sensor - Left -->
+  <gazebo reference="laser_left_link">
+    <sensor name="lidar_left" type="gpu_lidar">
       <always_on>true</always_on>
       <visualize>true</visualize>
       <topic>scan</topic>
       <update_rate>5</update_rate>
-      <gz_frame_id>laser_link</gz_frame_id>
+      <gz_frame_id>laser_left_link</gz_frame_id>
       <lidar>
         <scan>

Commit message: Swap laser link names and adjust visual orientation in URDF

File: src/sanad_description/urdf/sanad.urdf.xacro (robot description, xacro)
@@ -179,5 +179,5 @@
     <axis xyz="0 0 0" />
   </joint>
-  <link name="laser_right_link">
+  <link name="laser_left_link">
     <inertial>
       <origin xyz="-0.011945780406062 -0.000381929217680526 -0.0170649378129477" rpy="0 0 0" />
@@ -188,5 +188,5 @@
     </inertial>
     <visual>
-      <origin xyz="0 0 0" rpy="0 0 0" />
+      <origin xyz="0 0 0" rpy="1 1 1" />
       <geometry>
         <mesh filename="package://sanad_description/meshes/laser_link.STL" />
@@ -201,5 +201,5 @@
     </collision>
   </link>
-  <link name="laser_left_link">
+  <link name="laser_right_link">
     <inertial>
       <origin xyz="-0.011945780406062 -0.000381929217680526 -0.0170649378129477" rpy="0 0 0" />
@@ -223,14 +223,14 @@
     </collision>
   </link>
-  <joint name="laser_right_joint" type="fixed">
+  <joint name="laser_left_joint" type="fixed">
     <origin xyz="-0.265 ${-(0.245 +0.1)} 0.06" rpy="0 0 3.14" />
     <parent link="base_link" />
+    <child link="laser_left_link" />
+    <axis xyz="0 0 0" />
+  </joint>
+    <joint name="laser_right_joint" type="fixed">
+    <origin xyz="-0.265 ${(0.245 +0.1)} 0.06" rpy="0 0 3.14" />
+    <parent link="base_link" />
     <child link="laser_right_link" />
-    <axis xyz="0 0 0" />
-  </joint>
-    <joint name="laser_left_joint" type="fixed">
-    <origin xyz="-0.265 ${(0.245 +0.1)} 0.06" rpy="0 0 3.14" />
-    <parent link="base_link" />
-    <child link="laser_left_link" />
     <axis xyz="0 0 0" />
   </joint>

Commit message: Refactor URDF links and joints for wheelchair; add laser filters and update navigation launch configurations

File: src/sanad_description/urdf/sanad.urdf.xacro (robot description, xacro)
@@ -38,5 +38,5 @@
     <origin xyz="0 0 0.533" rpy="0 0 0"/>
   </joint>
-  <link name="wheel_right_link">
+  <link name="wheel_left_link">
     <inertial>
       <origin xyz="0 0 0" rpy="0 0 0" />
@@ -60,12 +60,12 @@
     </collision>
   </link>
-  <joint name="wheel_right_joint" type="continuous">
+  <joint name="wheel_left_joint" type="continuous">
     <origin xyz="0.22 -${0.580/2} -0.37" rpy="0 0 0" />
     <parent link="base_link" />
-    <child link="wheel_right_link" />
+    <child link="wheel_left_link" />
     <axis xyz="0 1 0" />
   </joint>
   <link
-    name="wheel_left_link">
+    name="wheel_right_link">
     <inertial>
       <origin xyz="0 0 0" rpy="0 0 0" />
@@ -89,8 +89,8 @@
     </collision>
   </link>
-  <joint name="wheel_left_joint" type="continuous">
+  <joint name="wheel_right_joint" type="continuous">
     <origin xyz="0.22 ${0.580/2} -0.37" rpy="0 0 0" />
     <parent link="base_link" />
-    <child link="wheel_left_link" />
+    <child link="wheel_right_link" />
     <axis xyz="0 1 0" />
   </joint>
@@ -188,5 +188,5 @@
     </inertial>
     <visual>
-      <origin xyz="0 0 0" rpy="1 1 1" />
+      <origin xyz="0 0 0" rpy="0 0 0" />
       <geometry>
         <mesh filename="package://sanad_description/meshes/laser_link.STL" />
@@ -224,5 +224,5 @@
   </link>
   <joint name="laser_left_joint" type="fixed">
-    <origin xyz="-0.265 ${-(0.245 +0.1)} 0.06" rpy="0 0 3.14" />
+    <origin xyz="-0.265 ${-(0.245 +0.1)} 0.06" rpy="0 0 1.57" />
     <parent link="base_link" />
     <child link="laser_left_link" />
@@ -230,5 +230,5 @@
   </joint>
     <joint name="laser_right_joint" type="fixed">
-    <origin xyz="-0.265 ${(0.245 +0.1)} 0.06" rpy="0 0 3.14" />
+    <origin xyz="-0.265 ${(0.245 +0.1)} 0.06" rpy="0 0 0" />
     <parent link="base_link" />
     <child link="laser_right_link" />
