Commit message: Adding Astra Depth Camera

File: src/sanad_description/urdf/sanad.urdf.xacro (robot description, xacro)
@@ -179,4 +179,32 @@
     <axis xyz="0 0 0" />
   </joint>
+  <link name="depth_camera_link">
+    <inertial>
+      <origin xyz="0 0 0" rpy="0 0 0" />
+      <mass value="0.1" />
+      <inertia ixx="0.0001" ixy="0.0" ixz="0.0"
+               iyy="0.0001" iyz="0.0"
+               izz="0.0001" />
+    </inertial>
+    <visual>
+      <origin xyz="0.02 0.025 0.045" rpy="1.57 0 1.57" />
+      <geometry>
+        <mesh filename="package://sanad_description/meshes/astra.stl" scale="0.001 0.001 0.001" />
+      </geometry>
+      <material name="dark_grey"/>
+    </visual>
+    <collision>
+      <origin xyz="0 0 0" rpy="0 0 0" />
+      <geometry>
+        <mesh filename="package://sanad_description/meshes/astra.stl" scale="0.001 0.001 0.001" />
+      </geometry>
+    </collision>
+  </link>
+  <joint name="depth_camera_joint" type="fixed">
+    <origin xyz="-0.32 -0.245 0.18" rpy="3.14 3.14 0" />
+    <parent link="base_link" />
+    <child link="depth_camera_link" />
+    <axis xyz="0 0 0" />
+  </joint>
   <link name="laser_left_link">
     <inertial>

File: src/sanad_description/urdf/sanad_gazebo.xacro (robot description, xacro)
@@ -111,4 +111,32 @@
           </linear_acceleration>
         </imu>
+    </sensor>
+  </gazebo>
+  <!-- RealSense RGB-D Camera -->
+  <gazebo reference="depth_camera_link">
+    <sensor name="realsense_d435" type="rgbd_camera">
+      <always_on>true</always_on>
+      <visualize>true</visualize>
+      <update_rate>30</update_rate>
+      <topic>realsense</topic>
+      <gz_frame_id>realsense_link</gz_frame_id>
+      <camera>
+        <horizontal_fov>1.3962634</horizontal_fov>
+        <image>
+          <width>640</width>
+          <height>480</height>
+          <format>R8G8B8</format>
+        </image>
+        <clip>
+          <near>0.1</near>
+          <far>10.0</far>
+        </clip>
+      </camera>
+      <depth_camera>
+        <clip>
+          <near>0.1</near>
+          <far>10.0</far>
+        </clip>
+      </depth_camera>
     </sensor>
   </gazebo>

Commit message: Update URDF and configuration files for wheelchair navigation; adjust laser joint positions, costmap parameters, and filter settings

File: src/sanad_description/urdf/sanad.urdf.xacro (robot description, xacro)
@@ -252,5 +252,5 @@
   </link>
   <joint name="laser_left_joint" type="fixed">
-    <origin xyz="-0.265 ${-(0.245 +0.1)} 0.06" rpy="0 0 1.57" />
+    <origin xyz="-0.265 ${-(0.245 +0.1)} -0.2" rpy="0 0 1.57" />
     <parent link="base_link" />
     <child link="laser_left_link" />
@@ -258,5 +258,5 @@
   </joint>
     <joint name="laser_right_joint" type="fixed">
-    <origin xyz="-0.265 ${(0.245 +0.1)} 0.06" rpy="0 0 0" />
+    <origin xyz="-0.265 ${(0.245 +0.1)} -0.2" rpy="0 0 0" />
     <parent link="base_link" />
     <child link="laser_right_link" />

Commit message: Fix wheel joint names and adjust orientations in URDF

File: src/sanad_description/urdf/sanad.urdf.xacro (robot description, xacro)
@@ -20,5 +20,5 @@
     </inertial>
     <visual>
-      <origin xyz="0 ${0.416/2} 0" rpy="0 0 0" />
+      <origin xyz="0 -${0.416/2} 0" rpy="0 0 3.14" />
       <geometry>
         <mesh filename="package://sanad_description/meshes/chase.stl" scale="0.001 0.001 0.001" />
@@ -27,5 +27,5 @@
     </visual>
     <collision>
-      <origin xyz="0 ${0.416/2} 0" rpy="0 0 0" />
+      <origin xyz="0 -${0.416/2} 0" rpy="0 0 0" />
       <geometry>
         <mesh filename="package://sanad_description/meshes/chase.stl" scale="0.001 0.001 0.001" />
@@ -33,9 +33,6 @@
     </collision>
   </link>
-  <joint name="base_joint" type="fixed">
-    <parent link="base_footprint"/>
-    <child link="base_link" />
-    <origin xyz="0 0 0.533" rpy="0 0 0"/>
-  </joint>
+  <!-- ^ Links Section -->
+  <!-- All link elements are grouped below -->
   <link name="wheel_left_link">
     <inertial>
@@ -60,10 +57,5 @@
     </collision>
   </link>
-  <joint name="wheel_left_joint" type="continuous">
-    <origin xyz="0.22 -${0.580/2} -0.37" rpy="0 0 0" />
-    <parent link="base_link" />
-    <child link="wheel_left_link" />
-    <axis xyz="0 1 0" />
-  </joint>
+  <!-- wheel_left_joint moved to Joints section -->
   <link
     name="wheel_right_link">
@@ -89,10 +81,5 @@
     </collision>
   </link>
-  <joint name="wheel_right_joint" type="continuous">
-    <origin xyz="0.22 ${0.580/2} -0.37" rpy="0 0 0" />
-    <parent link="base_link" />
-    <child link="wheel_right_link" />
-    <axis xyz="0 1 0" />
-  </joint>
+  <!-- wheel_right_joint moved to Joints section -->
   <link name="caster_front_link">
     <inertial>
@@ -117,10 +104,5 @@
     </collision>
   </link>
-  <joint name="caster_front_joint" type="fixed">
-    <origin xyz="-0.32 0.251 -0.44" rpy="1.57 1.57 0" />
-    <parent link="base_link" />
-    <child link="caster_front_link" />
-    <axis xyz="0 0 0" />
-  </joint>
+  <!-- caster_front_joint moved to Joints section -->
   <link name="caster_rear_link">
     <inertial>
@@ -145,10 +127,5 @@
     </collision>
   </link>
-  <joint name="caster_rear_joint" type="fixed">
-    <origin xyz="-0.32 -0.251 -0.44" rpy="1.57 1.57 0" />
-    <parent link="base_link" />
-    <child link="caster_rear_link" />
-    <axis xyz="0 0 0" />
-  </joint>
+  <!-- caster_rear_joint moved to Joints section -->
   <link name="imu_link">
     <inertial>
@@ -173,10 +150,5 @@
     </collision>
   </link>
-  <joint name="imu_joint" type="fixed">
-    <origin xyz="0 0 0.0698986241758014" rpy="0 0 0" />
-    <parent link="base_link" />
-    <child link="imu_link" />
-    <axis xyz="0 0 0" />
-  </joint>
+  <!-- imu_joint moved to Joints section -->
   <link name="depth_camera_link">
     <inertial>
@@ -201,10 +173,5 @@
     </collision>
   </link>
-  <joint name="depth_camera_joint" type="fixed">
-    <origin xyz="-0.32 -0.245 0.18" rpy="3.14 3.14 0" />
-    <parent link="base_link" />
-    <child link="depth_camera_link" />
-    <axis xyz="0 0 0" />
-  </joint>
+  <!-- depth_camera_joint moved to Joints section -->
   <link name="laser_left_link">
     <inertial>
@@ -251,12 +218,56 @@
     </collision>
   </link>
+  <!-- ^ Joints Section -->
+  <!-- All joint elements are grouped here -->
+  <joint name="base_joint" type="fixed">
+    <parent link="base_footprint"/>
+    <child link="base_link" />
+    <!-- ^Rotate base_link 180 degrees around Z so robot "front" is flipped -->
+    <origin xyz="0 0 0.533" rpy="0 0 0"/>
+  </joint>
+  <joint name="wheel_left_joint" type="continuous">
+    <origin xyz="-0.22 ${0.580/2} -0.37" rpy="0 0 0" />
+    <parent link="base_link" />
+    <child link="wheel_left_link" />
+    <axis xyz="0 1 0" />
+  </joint>
+  <joint name="wheel_right_joint" type="continuous">
+    <origin xyz="-0.22 -${0.580/2} -0.37" rpy="0 0 0" />
+    <parent link="base_link" />
+    <child link="wheel_right_link" />
+    <axis xyz="0 1 0" />
+  </joint>
+  <joint name="caster_front_joint" type="fixed">
+    <origin xyz="0.32 -0.251 -0.44" rpy="1.57 1.57 0" />
+    <parent link="base_link" />
+    <child link="caster_front_link" />
+    <axis xyz="0 0 0" />
+  </joint>
+  <joint name="caster_rear_joint" type="fixed">
+    <origin xyz="0.32 0.251 -0.44" rpy="1.57 1.57 0" />
+    <parent link="base_link" />
+    <child link="caster_rear_link" />
+    <axis xyz="0 0 0" />
+  </joint>
+  <joint name="imu_joint" type="fixed">
+    <origin xyz="0 0 0.0698986241758014" rpy="0 0 0" />
+    <parent link="base_link" />
+    <child link="imu_link" />
+    <axis xyz="0 0 0" />
+  </joint>
+  <joint name="depth_camera_joint" type="fixed">
+    <origin xyz="0.32 0.245 0.18" rpy="3.14 3.14 0" />
+    <parent link="base_link" />
+    <child link="depth_camera_link" />
+    <axis xyz="0 0 0" />
+  </joint>
   <joint name="laser_left_joint" type="fixed">
-    <origin xyz="-0.265 ${-(0.245 +0.1)} -0.2" rpy="0 0 1.57" />
+    <origin xyz="0.265 ${(0.245 +0.1)} -0.2" rpy="0 0 ${1.57 + 3.14}" />
     <parent link="base_link" />
     <child link="laser_left_link" />
     <axis xyz="0 0 0" />
   </joint>
-    <joint name="laser_right_joint" type="fixed">
-    <origin xyz="-0.265 ${(0.245 +0.1)} -0.2" rpy="0 0 0" />
+  <joint name="laser_right_joint" type="fixed">
+    <origin xyz="0.265 -${(0.245 +0.1)} -0.2" rpy="0 0 3.14" />
     <parent link="base_link" />
     <child link="laser_right_link" />

Commit message: Fix collision origin rotation for chase mesh in URDF

File: src/sanad_description/urdf/sanad.urdf.xacro (robot description, xacro)
@@ -27,5 +27,5 @@
     </visual>
     <collision>
-      <origin xyz="0 -${0.416/2} 0" rpy="0 0 0" />
+      <origin xyz="0 -${0.416/2} 0" rpy="0 0 3.14" />
       <geometry>
         <mesh filename="package://sanad_description/meshes/chase.stl" scale="0.001 0.001 0.001" />

Commit message: Update robot radius in costmap and planner server configurations to improve navigation accuracy

File: src/sanad_description/urdf/sanad.urdf.xacro (robot description, xacro)
@@ -153,5 +153,5 @@
   <link name="depth_camera_link">
     <inertial>
-      <origin xyz="0 0 0" rpy="0 0 0" />
+      <origin xyz="0.02 0.02 0.05" rpy="-1.57 3.14 4.71" />
       <mass value="0.1" />
       <inertia ixx="0.0001" ixy="0.0" ixz="0.0"
@@ -160,5 +160,5 @@
     </inertial>
     <visual>
-      <origin xyz="0.02 0.025 0.045" rpy="1.57 0 1.57" />
+      <origin xyz="0.02 0.02 0.05" rpy="-1.57 3.14 4.71" />
       <geometry>
         <mesh filename="package://sanad_description/meshes/astra.stl" scale="0.001 0.001 0.001" />
@@ -167,5 +167,5 @@
     </visual>
     <collision>
-      <origin xyz="0 0 0" rpy="0 0 0" />
+      <origin xyz="0.02 0.02 0.05" rpy="-1.57 3.14 4.71" />
       <geometry>
         <mesh filename="package://sanad_description/meshes/astra.stl" scale="0.001 0.001 0.001" />
@@ -176,5 +176,5 @@
   <link name="laser_left_link">
     <inertial>
-      <origin xyz="-0.011945780406062 -0.000381929217680526 -0.0170649378129477" rpy="0 0 0" />
+      <origin xyz="-0.011945780406062 -0.000381929217680526 -0.0170649378129477" rpy="0 0 ${1.57 + 3.14}" />
       <mass value="0.073084435549317" />
       <inertia ixx="1.96074931730795E-05" ixy="-3.62091076640009E-07" ixz="4.28230084046735E-07"
@@ -183,5 +183,5 @@
     </inertial>
     <visual>
-      <origin xyz="0 0 0" rpy="0 0 0" />
+      <origin xyz="0 0 0" rpy="0 0 ${1.57 + 3.14}" />
       <geometry>
         <mesh filename="package://sanad_description/meshes/laser_link.STL" />
@@ -190,5 +190,5 @@
     </visual>
     <collision>
-      <origin xyz="0 0 0" rpy="0 0 0" />
+      <origin xyz="0 0 0" rpy="0 0 ${1.57 + 3.14}" />
       <geometry>
         <mesh filename="package://sanad_description/meshes/laser_link.STL" />
@@ -198,5 +198,5 @@
   <link name="laser_right_link">
     <inertial>
-      <origin xyz="-0.011945780406062 -0.000381929217680526 -0.0170649378129477" rpy="0 0 0" />
+      <origin xyz="-0.011945780406062 -0.000381929217680526 -0.0170649378129477" rpy="0 0 ${1.57 + 3.14}" />
       <mass value="0.073084435549317" />
       <inertia ixx="1.96074931730795E-05" ixy="-3.62091076640009E-07" ixz="4.28230084046735E-07"
@@ -205,5 +205,5 @@
     </inertial>
     <visual>
-      <origin xyz="0 0 0" rpy="0 0 0" />
+      <origin xyz="0 0 0" rpy="0 0 ${1.57 + 3.14}" />
       <geometry>
         <mesh filename="package://sanad_description/meshes/laser_link.STL" />
@@ -212,5 +212,5 @@
     </visual>
     <collision>
-      <origin xyz="0 0 0" rpy="0 0 0" />
+      <origin xyz="0 0 0" rpy="0 0 ${1.57 + 3.14}" />
       <geometry>
         <mesh filename="package://sanad_description/meshes/laser_link.STL" />
@@ -223,5 +223,4 @@
     <parent link="base_footprint"/>
     <child link="base_link" />
-    <!-- ^Rotate base_link 180 degrees around Z so robot "front" is flipped -->
     <origin xyz="0 0 0.533" rpy="0 0 0"/>
   </joint>
@@ -257,5 +256,5 @@
   </joint>
   <joint name="depth_camera_joint" type="fixed">
-    <origin xyz="0.32 0.245 0.18" rpy="3.14 3.14 0" />
+    <origin xyz="0.3 0.24 0.23" rpy="0 0 0" />
     <parent link="base_link" />
     <child link="depth_camera_link" />
@@ -263,5 +262,5 @@
   </joint>
   <joint name="laser_left_joint" type="fixed">
-    <origin xyz="0.265 ${(0.245 +0.1)} -0.2" rpy="0 0 ${1.57 + 3.14}" />
+    <origin xyz="0.265 ${(0.245 +0.1)} -0.2" rpy="0 0 ${3.14 + 1.57}" />
     <parent link="base_link" />
     <child link="laser_left_link" />

Commit message: checkpoint

File: src/sanad_description/urdf/sanad.urdf.xacro (robot description, xacro)
@@ -268,5 +268,5 @@
   </joint>
   <joint name="laser_right_joint" type="fixed">
-    <origin xyz="0.265 -${(0.245 +0.1)} -0.2" rpy="0 0 3.14" />
+    <origin xyz="0.265 -${(0.245 +0.1)} -0.2" rpy="0 0 1.57" />
     <parent link="base_link" />
     <child link="laser_right_link" />

Commit message: Update Lidar configurations and add Google Cloud setup documentation
- Enable angle cropping for Lidar with updated min/max values in real_robot.launch.py
- Adjust laser_left_joint orientation in sanand.urdf.xacro
- Comment out unused parameters in laser_left_filter.yaml and laser_right_filter.yaml
- Comment out navigation components in navigation.launch.py
- Add Google Cloud setup guide for Gemini on Vertex AI

File: src/sanad_description/urdf/sanad.urdf.xacro (robot description, xacro)
@@ -262,5 +262,5 @@
   </joint>
   <joint name="laser_left_joint" type="fixed">
-    <origin xyz="0.265 ${(0.245 +0.1)} -0.2" rpy="0 0 ${3.14 + 1.57}" />
+    <origin xyz="0.265 ${(0.245 +0.1)} -0.2" rpy="0 0 1.57" />
     <parent link="base_link" />
     <child link="laser_left_link" />

Commit message: fixing real lidar positions

File: src/sanad_description/urdf/sanad.urdf.xacro (robot description, xacro)
@@ -262,5 +262,5 @@
   </joint>
   <joint name="laser_left_joint" type="fixed">
-    <origin xyz="0.265 ${(0.245 +0.1)} -0.2" rpy="0 0 1.57" />
+    <origin xyz="0.265 ${(0.245 +0.035)} -0.2" rpy="0 0 1.57" />
     <parent link="base_link" />
     <child link="laser_left_link" />
@@ -268,5 +268,5 @@
   </joint>
   <joint name="laser_right_joint" type="fixed">
-    <origin xyz="0.265 -${(0.245 +0.1)} -0.2" rpy="0 0 1.57" />
+    <origin xyz="0.265 -${(0.245 +0.035)} -0.2" rpy="0 0 1.57" />
     <parent link="base_link" />
     <child link="laser_right_link" />
