Commit message: Add camera node and update launch configurations for simulation and real scenarios

File: src/sanad_description/urdf/sanad.urdf.xacro (robot description, xacro)
@@ -151,5 +151,5 @@
   </link>
   <!-- imu_joint moved to Joints section -->
-  <link name="depth_camera_link">
+  <link name="camera_link">
     <inertial>
       <origin xyz="0.02 0.02 0.05" rpy="-1.57 3.14 4.71" />
@@ -173,5 +173,5 @@
     </collision>
   </link>
-  <!-- depth_camera_joint moved to Joints section -->
+  <!-- camera_joint moved to Joints section -->
   <link name="laser_left_link">
     <inertial>
@@ -218,4 +218,16 @@
     </collision>
   </link>
+  <xacro:if value="$(arg is_sim)">
+    <xacro:property name="laser_left_y" value="${0.245 + 0.1}" />
+    <xacro:property name="laser_right_y" value="-${0.245 + 0.1}" />
+    <xacro:property name="laser_left_yaw" value="${3.14 + 1.57}" />
+    <xacro:property name="laser_right_yaw" value="3.14" />
+  </xacro:if>
+  <xacro:unless value="$(arg is_sim)">
+    <xacro:property name="laser_left_y" value="${0.245 + 0.035}" />
+    <xacro:property name="laser_right_y" value="-${0.245 + 0.035}" />
+    <xacro:property name="laser_left_yaw" value="1.57" />
+    <xacro:property name="laser_right_yaw" value="1.57" />
+  </xacro:unless>
   <!-- ^ Joints Section -->
   <!-- All joint elements are grouped here -->
@@ -255,12 +267,12 @@
     <axis xyz="0 0 0" />
   </joint>
-  <joint name="depth_camera_joint" type="fixed">
+  <joint name="camera_joint" type="fixed">
     <origin xyz="0.3 0.24 0.23" rpy="0 0 0" />
     <parent link="base_link" />
-    <child link="depth_camera_link" />
+    <child link="camera_link" />
     <axis xyz="0 0 0" />
   </joint>
   <joint name="laser_left_joint" type="fixed">
-    <origin xyz="0.265 ${(0.245 +0.035)} -0.2" rpy="0 0 1.57" />
+    <origin xyz="0.265 ${laser_left_y} -0.2" rpy="0 0 ${laser_left_yaw}" />
     <parent link="base_link" />
     <child link="laser_left_link" />
@@ -268,5 +280,5 @@
   </joint>
   <joint name="laser_right_joint" type="fixed">
-    <origin xyz="0.265 -${(0.245 +0.035)} -0.2" rpy="0 0 1.57" />
+    <origin xyz="0.265 ${laser_right_y} -0.2" rpy="0 0 ${laser_right_yaw}" />
     <parent link="base_link" />
     <child link="laser_right_link" />

Commit message: feat: add simulation-specific laser sensor configurations and launch filters for improved navigation accuracy

File: src/sanad_description/urdf/sanad.urdf.xacro (robot description, xacro)
@@ -261,16 +261,32 @@
     <axis xyz="0 0 0" />
   </joint>
-  <joint name="laser_left_joint" type="fixed">
-    <origin xyz="0.265 ${(0.245 +0.035)} -0.2" rpy="0 0 1.57" />
-    <parent link="base_link" />
-    <child link="laser_left_link" />
-    <axis xyz="0 0 0" />
-  </joint>
-  <joint name="laser_right_joint" type="fixed">
-    <origin xyz="0.265 -${(0.245 +0.035)} -0.2" rpy="0 0 1.57" />
-    <parent link="base_link" />
-    <child link="laser_right_link" />
-    <axis xyz="0 0 0" />
-  </joint>
+  <xacro:if value="$(arg is_sim)">
+    <joint name="laser_left_joint" type="fixed">
+      <origin xyz="0.265 ${(0.245 +0.1)} -0.2" rpy="0 0 ${3.14 + 1.57}" />
+      <parent link="base_link" />
+      <child link="laser_left_link" />
+      <axis xyz="0 0 0" />
+    </joint>
+    <joint name="laser_right_joint" type="fixed">
+      <origin xyz="0.265 -${(0.245 +0.1)} -0.2" rpy="0 0 3.14" />
+      <parent link="base_link" />
+      <child link="laser_right_link" />
+      <axis xyz="0 0 0" />
+    </joint>
+  </xacro:if>
+  <xacro:unless value="$(arg is_sim)">
+    <joint name="laser_left_joint" type="fixed">
+      <origin xyz="0.265 ${(0.245 +0.035)} -0.2" rpy="0 0 1.57" />
+      <parent link="base_link" />
+      <child link="laser_left_link" />
+      <axis xyz="0 0 0" />
+    </joint>
+    <joint name="laser_right_joint" type="fixed">
+      <origin xyz="0.265 -${(0.245 +0.035)} -0.2" rpy="0 0 1.57" />
+      <parent link="base_link" />
+      <child link="laser_right_link" />
+      <axis xyz="0 0 0" />
+    </joint>
+  </xacro:unless>
   <material name="blue">
     <color rgba="0 0 1 1"/>
